File: DSAT_Telemetry_Board/DSAT_Telemetry_Board/USBC.kicad_sch (KiCad schematic)
At the start: 3 parts

Commit message: Updated Microcontroller Pinout Names
Updated Names
Connections:
- net D+ is gone; now on net GND: USB?.6 (DP1), USB?.8 (DP2)
Other:
- moved on the sheet: R?, USB?

Commit message: Seperate Branch
Updated Pin names, Added LNA, Fixed Pins on USB connection
Connections:
- net GND: no longer USB?.6 (DP1), USB?.8 (DP2)
- new net D+: USB?.6 (DP1), USB?.8 (DP2)
Changed lines of the file:
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@@
   (junction (at 144.78 92.71) (diameter 0) (color 0 0 0 0)
-  )
-  (junction (at 148.59 102.87) (diameter 0) (color 0 0 0 0)
   )
   (junction (at 135.89 118.11) (diameter 0) (color 0 0 0 0)
@@
     (stroke (width 0) (type default) (color 0 0 0 0))
   )
-  (wire (pts (xy 148.59 102.87) (xy 154.94 102.87))
-    (stroke (width 0) (type default) (color 0 0 0 0))
-  )
   (wire (pts (xy 129.54 92.71) (xy 144.78 92.71))
     (stroke (width 0) (type default) (color 0 0 0 0))
   )
-  (wire (pts (xy 130.81 106.68) (xy 156.21 106.68))
+  (wire (pts (xy 130.81 106.68) (xy 158.75 106.68))
     (stroke (width 0) (type default) (color 0 0 0 0))
   )
@@
     (stroke (width 0) (type default) (color 0 0 0 0))
   )
-  (wire (pts (xy 134.62 102.87) (xy 148.59 102.87))
+  (wire (pts (xy 134.62 102.87) (xy 158.75 102.87))
     (stroke (width 0) (type default) (color 0 0 0 0))
   )
-  (global_label "D-" (shape input) (at 156.21 106.68 0) (fields_autoplaced)
+  (hierarchical_label "D+" (shape input) (at 158.75 102.87 0)
     (effects (font (size 1.27 1.27)) (justify left))
-    (property "Intersheet References" "${INTERSHEET_REFS}" (id 0) (at 161.4655 106.6006 0)
-      (effects (font (size 1.27 1.27)) (justify left) hide)
-    )
   )
-  (global_label "D+" (shape input) (at 154.94 102.87 0) (fields_autoplaced)
+  (hierarchical_label "D-" (shape input) (at 158.75 106.68 0)
     (effects (font (size 1.27 1.27)) (justify left))
-    (property "Intersheet References" "${INTERSHEET_REFS}" (id 0) (at 160.1955 102.7906 0)
-      (effects (font (size 1.27 1.27)) (justify left) hide)
-    )
   )
   (symbol (lib_id "Type-C:HRO-TYPE-C-31-M-12") (at 127 104.14 0) (unit 1)
