File: DSAT_Telemetry_Board/DSAT_Telemetry_Board/USBC.kicad_sch (KiCad schematic)
At the start: 3 parts

Commit message: Added Watchdog Timer
Connections:
- net GND: no longer USB?.6 (DP1), USB?.8 (DP2)
- new net D+: USB?.6 (DP1), USB?.8 (DP2)
Changed lines of the file:
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@@
   (junction (at 144.78 92.71) (diameter 0) (color 0 0 0 0)
-  )
-  (junction (at 148.59 102.87) (diameter 0) (color 0 0 0 0)
   )
   (junction (at 135.89 118.11) (diameter 0) (color 0 0 0 0)
@@
     (stroke (width 0) (type default) (color 0 0 0 0))
   )
-  (wire (pts (xy 148.59 102.87) (xy 154.94 102.87))
-    (stroke (width 0) (type default) (color 0 0 0 0))
-  )
   (wire (pts (xy 129.54 92.71) (xy 144.78 92.71))
     (stroke (width 0) (type default) (color 0 0 0 0))
@@
     (stroke (width 0) (type default) (color 0 0 0 0))
   )
-  (wire (pts (xy 134.62 102.87) (xy 148.59 102.87))
+  (wire (pts (xy 134.62 102.87) (xy 154.94 102.87))
     (stroke (width 0) (type default) (color 0 0 0 0))
   )

Commit message: More footprints
Parts:
- R? (x2): footprint Resistor_SMD:R_0805_2012Metric_Pad1.20x1.40mm_HandSolder -> Resistor_SMD:R_0805_2012Metric
Changed lines of the file:
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@@
       (effects (font (size 1.27 1.27)) (justify left))
     )
-    (property "Footprint" "Resistor_SMD:R_0805_2012Metric_Pad1.20x1.40mm_HandSolder" (id 2) (at 148.59 100.33 0)
+    (property "Footprint" "Resistor_SMD:R_0805_2012Metric" (id 2) (at 148.59 100.33 0)
       (effects (font (size 1.27 1.27)) hide)
     )
-    (property "Datasheet" "~" (id 3) (at 148.59 100.33 0)
+    (property "Datasheet" "https://www.digikey.com/en/products/detail/panasonic-electronic-components/ERA-6ARW512V/3073815" (id 3) (at 148.59 100.33 0)
       (effects (font (size 1.27 1.27)) hide)
     )
@@
       (effects (font (size 1.27 1.27)) (justify left))
     )
-    (property "Footprint" "Resistor_SMD:R_0805_2012Metric_Pad1.20x1.40mm_HandSolder" (id 2) (at 138.43 107.95 0)
+    (property "Footprint" "Resistor_SMD:R_0805_2012Metric" (id 2) (at 138.43 107.95 0)
       (effects (font (size 1.27 1.27)) hide)
     )
-    (property "Datasheet" "~" (id 3) (at 138.43 107.95 0)
+    (property "Datasheet" "https://www.digikey.com/en/products/detail/panasonic-electronic-components/ERA-6ARW512V/3073815" (id 3) (at 138.43 107.95 0)
       (effects (font (size 1.27 1.27)) hide)
     )

Commit message: RX_SWitch, test points
Parts:
- R? (x2): footprint Resistor_SMD:R_0805_2012Metric -> Resistor_SMD:R_0402_1005Metric_Pad0.72x0.64mm_HandSolder
Changed lines of the file:
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@@
     )
   )
-  (symbol (lib_id "Type-C:HRO-TYPE-C-31-M-12") (at 127 104.14 0) (unit 1)
+  (symbol (lib_id "Type-C:HRO-TYPE-C-31-M-12") (at 127 104.14 0)
     (in_bom yes) (on_board yes) (fields_autoplaced)
     (property "Reference" "USB?" (id 0) (at 121.285 83.82 0)
@@
     (pin "9")
   )
-  (symbol (lib_id "power:VCC") (at 146.05 92.71 270) (unit 1)
+  (symbol (lib_id "power:VCC") (at 146.05 92.71 270)
     (in_bom yes) (on_board yes) (fields_autoplaced)
     (property "Reference" "#PWR?" (id 0) (at 142.24 92.71 0)
@@
     (pin "1")
   )
-  (symbol (lib_id "power:GND") (at 135.89 123.19 0) (unit 1)
+  (symbol (lib_id "power:GND") (at 135.89 123.19 0)
     (in_bom yes) (on_board yes) (fields_autoplaced)
     (property "Reference" "#PWR?" (id 0) (at 135.89 129.54 0)
@@
     (pin "1")
   )
-  (symbol (lib_id "Device:R_Small") (at 148.59 100.33 0) (unit 1)
+  (symbol (lib_id "Device:R_Small") (at 148.59 100.33 0)
     (in_bom yes) (on_board yes) (fields_autoplaced)
     (property "Reference" "R?" (id 0) (at 151.13 99.0599 0)
@@
       (effects (font (size 1.27 1.27)) (justify left))
     )
-    (property "Footprint" "Resistor_SMD:R_0805_2012Metric" (id 2) (at 148.59 100.33 0)
+    (property "Footprint" "Resistor_SMD:R_0402_1005Metric_Pad0.72x0.64mm_HandSolder" (id 2) (at 148.59 100.33 0)
       (effects (font (size 1.27 1.27)) hide)
     )
@@
     (pin "2")
   )
-  (symbol (lib_id "Device:R_Small") (at 138.43 107.95 0) (unit 1)
+  (symbol (lib_id "Device:R_Small") (at 138.43 107.95 0)
     (in_bom yes) (on_board yes) (fields_autoplaced)
     (property "Reference" "R?" (id 0) (at 140.97 106.6799 0)
@@
       (effects (font (size 1.27 1.27)) (justify left))
     )
-    (property "Footprint" "Resistor_SMD:R_0805_2012Metric" (id 2) (at 138.43 107.95 0)
+    (property "Footprint" "Resistor_SMD:R_0402_1005Metric_Pad0.72x0.64mm_HandSolder" (id 2) (at 138.43 107.95 0)
       (effects (font (size 1.27 1.27)) hide)
     )

Commit message: RX_SWitch, test points
Parts:
- gave numbers to parts that had none: 3
Connections:
- net D+ renamed USB_D+
- net D- renamed USB_D-
- net VCC renamed +3.3V
Changed lines of the file:
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@@
     (stroke (width 0) (type default) (color 0 0 0 0))
   )
-  (global_label "D-" (shape input) (at 156.21 106.68 0) (fields_autoplaced)
+  (hierarchical_label "USB_D+" (shape input) (at 154.94 102.87 0)
     (effects (font (size 1.27 1.27)) (justify left))
-    (property "Intersheet References" "${INTERSHEET_REFS}" (id 0) (at 161.4655 106.6006 0)
-      (effects (font (size 1.27 1.27)) (justify left) hide)
-    )
   )
-  (global_label "D+" (shape input) (at 154.94 102.87 0) (fields_autoplaced)
+  (hierarchical_label "USB_D-" (shape input) (at 156.21 106.68 0)
     (effects (font (size 1.27 1.27)) (justify left))
-    (property "Intersheet References" "${INTERSHEET_REFS}" (id 0) (at 160.1955 102.7906 0)
-      (effects (font (size 1.27 1.27)) (justify left) hide)
-    )
   )
-  (symbol (lib_id "Type-C:HRO-TYPE-C-31-M-12") (at 127 104.14 0)
+  (symbol (lib_id "Type-C:HRO-TYPE-C-31-M-12") (at 127 104.14 0) (unit 1)
     (in_bom yes) (on_board yes) (fields_autoplaced)
-    (property "Reference" "USB?" (id 0) (at 121.285 83.82 0)
+    (property "Reference" "USB1" (id 0) (at 121.285 83.82 0)
       (effects (font (size 1.524 1.524)))
     )
@@
     (pin "9")
   )
-  (symbol (lib_id "power:VCC") (at 146.05 92.71 270)
+  (symbol (lib_id "power:+3.3V") (at 146.05 92.71 270) (unit 1)
     (in_bom yes) (on_board yes) (fields_autoplaced)
-    (property "Reference" "#PWR?" (id 0) (at 142.24 92.71 0)
+    (property "Reference" "#PWR0146" (id 0) (at 142.24 92.71 0)
       (effects (font (size 1.27 1.27)) hide)
     )
-    (property "Value" "VCC" (id 1) (at 149.86 92.7099 90)
+    (property "Value" "+3.3V" (id 1) (at 149.86 92.7099 90)
       (effects (font (size 1.27 1.27)) (justify left))
     )
@@
     (pin "1")
   )
-  (symbol (lib_id "power:GND") (at 135.89 123.19 0)
+  (symbol (lib_id "power:GND") (at 135.89 123.19 0) (unit 1)
     (in_bom yes) (on_board yes) (fields_autoplaced)
-    (property "Reference" "#PWR?" (id 0) (at 135.89 129.54 0)
+    (property "Reference" "#PWR0145" (id 0) (at 135.89 129.54 0)
       (effects (font (size 1.27 1.27)) hide)
     )
@@
     (pin "1")
   )
-  (symbol (lib_id "Device:R_Small") (at 148.59 100.33 0)
+  (symbol (lib_id "Device:R_Small") (at 148.59 100.33 0) (unit 1)
     (in_bom yes) (on_board yes) (fields_autoplaced)
-    (property "Reference" "R?" (id 0) (at 151.13 99.0599 0)
+    (property "Reference" "R13" (id 0) (at 151.13 99.0599 0)
       (effects (font (size 1.27 1.27)) (justify left))
     )
@@
     (pin "2")
   )
-  (symbol (lib_id "Device:R_Small") (at 138.43 107.95 0)
+  (symbol (lib_id "Device:R_Small") (at 138.43 107.95 0) (unit 1)
     (in_bom yes) (on_board yes) (fields_autoplaced)
-    (property "Reference" "R?" (id 0) (at 140.97 106.6799 0)
+    (property "Reference" "R12" (id 0) (at 140.97 106.6799 0)
       (effects (font (size 1.27 1.27)) (justify left))
     )

Commit message: Layout halfway done
Connections:
- net +3.3V renamed VBUS
- no-connect marks 0 -> 2
Changed lines of the file:
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@@
   (junction (at 134.62 102.87) (diameter 0) (color 0 0 0 0)
   )
+  (no_connect (at 129.54 95.25))
+  (no_connect (at 129.54 110.49))
   (wire (pts (xy 134.62 107.95) (xy 134.62 102.87))
     (stroke (width 0) (type default) (color 0 0 0 0))
@@
     (pin "9")
   )
-  (symbol (lib_id "power:+3.3V") (at 146.05 92.71 270) (unit 1)
-    (in_bom yes) (on_board yes) (fields_autoplaced)
-    (property "Reference" "#PWR0146" (id 0) (at 142.24 92.71 0)
-      (effects (font (size 1.27 1.27)) hide)
-    )
-    (property "Value" "+3.3V" (id 1) (at 149.86 92.7099 90)
-      (effects (font (size 1.27 1.27)) (justify left))
-    )
-    (property "Footprint" "" (id 2) (at 146.05 92.71 0)
-      (effects (font (size 1.27 1.27)) hide)
-    )
-    (property "Datasheet" "" (id 3) (at 146.05 92.71 0)
-      (effects (font (size 1.27 1.27)) hide)
-    )
-    (pin "1")
-  )
   (symbol (lib_id "power:GND") (at 135.89 123.19 0) (unit 1)
     (in_bom yes) (on_board yes) (fields_autoplaced)
@@
       (effects (font (size 1.27 1.27)) hide)
     )
+    (pin "1")
+  )
+  (symbol (lib_id "power:VBUS") (at 146.05 92.71 0) (unit 1)
+    (in_bom yes) (on_board yes) (fields_autoplaced)
+    (property "Reference" "#PWR0146" (id 0) (at 146.05 96.52 0)
+      (effects (font (size 1.27 1.27)) hide)
+    )
+    (property "Value" "VBUS" (id 1) (at 146.05 87.63 0))
+    (property "Footprint" "" (id 2) (at 146.05 92.71 0)
+      (effects (font (size 1.27 1.27)) hide)
+    )
+    (property "Datasheet" "" (id 3) (at 146.05 92.71 0)
+      (effects (font (size 1.27 1.27)) hide)
+    )
