File: DSAT_Telemetry_Board/DSAT_Telemetry_Board/Microcontroller.kicad_sch (KiCad schematic)
At the start: 20 parts

Commit message: Some footprints
Parts:
- C? (x11): footprint (none) -> Capacitor_SMD:C_0201_0603Metric
- R?: footprint (none) -> Resistor_SMD:R_0402_1005Metric
Changed lines of the file:
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@@
       (effects (font (size 1.27 1.27)) (justify left))
     )
-    (property "Footprint" "" (id 2) (at 152.7048 36.83 0)
-      (effects (font (size 1.27 1.27)) hide)
-    )
-    (property "Datasheet" "~" (id 3) (at 153.67 33.02 0)
+    (property "Footprint" "Capacitor_SMD:C_0201_0603Metric" (id 2) (at 152.7048 36.83 0)
+      (effects (font (size 1.27 1.27)) hide)
+    )
+    (property "Datasheet" "https://www.digikey.com/en/products/detail/murata-electronics/GRM033R60J105MEA2D/4213369" (id 3) (at 153.67 33.02 0)
       (effects (font (size 1.27 1.27)) hide)
     )
@@
       (effects (font (size 1.27 1.27)) (justify left))
     )
-    (property "Footprint" "" (id 2) (at 132.3848 36.83 0)
-      (effects (font (size 1.27 1.27)) hide)
-    )
-    (property "Datasheet" "~" (id 3) (at 133.35 33.02 0)
+    (property "Footprint" "Capacitor_SMD:C_0201_0603Metric" (id 2) (at 132.3848 36.83 0)
+      (effects (font (size 1.27 1.27)) hide)
+    )
+    (property "Datasheet" "https://www.digikey.com/en/products/detail/murata-electronics/GRM033R60J105MEA2D/4213369" (id 3) (at 133.35 33.02 0)
       (effects (font (size 1.27 1.27)) hide)
     )
@@
       (effects (font (size 1.27 1.27)) (justify left))
     )
-    (property "Footprint" "" (id 2) (at 191.4652 36.83 0)
-      (effects (font (size 1.27 1.27)) hide)
-    )
-    (property "Datasheet" "~" (id 3) (at 190.5 33.02 0)
+    (property "Footprint" "Capacitor_SMD:C_0201_0603Metric" (id 2) (at 191.4652 36.83 0)
+      (effects (font (size 1.27 1.27)) hide)
+    )
+    (property "Datasheet" "https://www.digikey.com/en/products/detail/murata-electronics/GRM033C71C104KE14D/5027472" (id 3) (at 190.5 33.02 0)
       (effects (font (size 1.27 1.27)) hide)
     )
@@
       (effects (font (size 1.27 1.27)) (justify left))
     )
-    (property "Footprint" "" (id 2) (at 246.0752 36.83 0)
-      (effects (font (size 1.27 1.27)) hide)
-    )
-    (property "Datasheet" "~" (id 3) (at 245.11 33.02 0)
+    (property "Footprint" "Capacitor_SMD:C_0201_0603Metric" (id 2) (at 246.0752 36.83 0)
+      (effects (font (size 1.27 1.27)) hide)
+    )
+    (property "Datasheet" "https://www.digikey.com/en/products/detail/murata-electronics/GRM033R60J105MEA2D/4213369" (id 3) (at 245.11 33.02 0)
       (effects (font (size 1.27 1.27)) hide)
     )
@@
       (effects (font (size 1.27 1.27)) (justify left))
     )
-    (property "Footprint" "" (id 2) (at 200.3552 57.15 0)
-      (effects (font (size 1.27 1.27)) hide)
-    )
-    (property "Datasheet" "~" (id 3) (at 199.39 53.34 0)
+    (property "Footprint" "Capacitor_SMD:C_0201_0603Metric" (id 2) (at 200.3552 57.15 0)
+      (effects (font (size 1.27 1.27)) hide)
+    )
+    (property "Datasheet" "https://www.digikey.com/en/products/detail/murata-electronics/GRM033C71C104KE14D/5027472" (id 3) (at 199.39 53.34 0)
       (effects (font (size 1.27 1.27)) hide)
     )
@@
       (effects (font (size 1.27 1.27)) (justify right))
     )
-    (property "Footprint" "" (id 2) (at 213.0552 80.01 0)
-      (effects (font (size 1.27 1.27)) hide)
-    )
-    (property "Datasheet" "~" (id 3) (at 212.09 83.82 0)
+    (property "Footprint" "Capacitor_SMD:C_0201_0603Metric" (id 2) (at 213.0552 80.01 0)
+      (effects (font (size 1.27 1.27)) hide)
+    )
+    (property "Datasheet" "https://www.digikey.com/en/products/detail/murata-electronics/GRM0335C1H100FA01J/4358681" (id 3) (at 212.09 83.82 0)
       (effects (font (size 1.27 1.27)) hide)
     )
@@
       (effects (font (size 1.27 1.27)) (justify left))
     )
-    (property "Footprint" "" (id 2) (at 205.4352 36.83 0)
-      (effects (font (size 1.27 1.27)) hide)
-    )
-    (property "Datasheet" "~" (id 3) (at 204.47 33.02 0)
+    (property "Footprint" "Capacitor_SMD:C_0201_0603Metric" (id 2) (at 205.4352 36.83 0)
+      (effects (font (size 1.27 1.27)) hide)
+    )
+    (property "Datasheet" "https://www.digikey.com/en/products/detail/murata-electronics/GRM033C71C104KE14D/5027472" (id 3) (at 204.47 33.02 0)
       (effects (font (size 1.27 1.27)) hide)
     )
@@
     (property "Reference" "R?" (id 0) (at 218.44 104.14 90))
     (property "Value" "10kOhm" (id 1) (at 218.44 106.68 90))
-    (property "Footprint" "" (id 2) (at 218.44 103.378 90)
-      (effects (font (size 1.27 1.27)) hide)
-    )
-    (property "Datasheet" "~" (id 3) (at 218.44 101.6 0)
+    (property "Footprint" "Resistor_SMD:R_0402_1005Metric" (id 2) (at 218.44 103.378 90)
+      (effects (font (size 1.27 1.27)) hide)
+    )
+    (property "Datasheet" "https://www.digikey.com/en/products/detail/yageo/RC0402JR-1310KL/13694115" (id 3) (at 218.44 101.6 0)
       (effects (font (size 1.27 1.27)) hide)
     )
@@
       (effects (font (size 1.27 1.27)) (justify left))
     )
-    (property "Footprint" "" (id 2) (at 164.1348 36.83 0)
-      (effects (font (size 1.27 1.27)) hide)
-    )
-    (property "Datasheet" "~" (id 3) (at 165.1 33.02 0)
+    (property "Footprint" "Capacitor_SMD:C_0201_0603Metric" (id 2) (at 164.1348 36.83 0)
+      (effects (font (size 1.27 1.27)) hide)
+    )
+    (property "Datasheet" "https://www.digikey.com/en/products/detail/murata-electronics/GRM033C80J123KE01D/2543438" (id 3) (at 165.1 33.02 0)
       (effects (font (size 1.27 1.27)) hide)
     )
@@
       (effects (font (size 1.27 1.27)) (justify left))
     )
-    (property "Footprint" "" (id 2) (at 232.1052 36.83 0)
-      (effects (font (size 1.27 1.27)) hide)
-    )
-    (property "Datasheet" "~" (id 3) (at 231.14 33.02 0)
+    (property "Footprint" "Capacitor_SMD:C_0201_0603Metric" (id 2) (at 232.1052 36.83 0)
+      (effects (font (size 1.27 1.27)) hide)
+    )
+    (property "Datasheet" "https://www.digikey.com/en/products/detail/murata-electronics/GRM033C71C104KE14D/5027472" (id 3) (at 231.14 33.02 0)
       (effects (font (size 1.27 1.27)) hide)
     )
@@
       (effects (font (size 1.27 1.27)) (justify left))
     )
-    (property "Footprint" "" (id 2) (at 240.9952 87.63 0)
-      (effects (font (size 1.27 1.27)) hide)
-    )
-    (property "Datasheet" "~" (id 3) (at 240.03 83.82 0)
+    (property "Footprint" "Capacitor_SMD:C_0201_0603Metric" (id 2) (at 240.9952 87.63 0)
+      (effects (font (size 1.27 1.27)) hide)
+    )
+    (property "Datasheet" "https://www.digikey.com/en/products/detail/murata-electronics/GRM0335C1H100FA01J/4358681" (id 3) (at 240.03 83.82 0)
       (effects (font (size 1.27 1.27)) hide)
     )
@@
       (effects (font (size 1.27 1.27)) (justify left))
     )
-    (property "Footprint" "" (id 2) (at 219.4052 36.83 0)
-      (effects (font (size 1.27 1.27)) hide)
-    )
-    (property "Datasheet" "~" (id 3) (at 218.44 33.02 0)
-      (effects (font (size 1.27 1.27)) hide)
-    )
+    (property "Footprint" "Capacitor_SMD:C_0201_0603Metric" (id 2) (at 219.4052 36.83 0)
+      (effects (font (size 1.27 1.27)) hide)
+    )
+    (property "Datasheet" "https://www.digikey.com/en/products/detail/murata-electronics/GRM033C71C104KE14D/5027472" (id 3) (at 218.44 33.02 0)
+      (effects (font (size 1.27 1.27)) hide)
+    )
