File: DSAT_Telemetry_Board/DSAT_Telemetry_Board/TX_Transcieiver.kicad_sch (KiCad schematic)
At the start: 15 parts

Commit message: More footprints
Parts:
- C? (x7): footprint (none) -> Capacitor_SMD:C_0201_0603Metric
Changed lines of the file:
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@@
       (effects (font (size 1.27 1.27)) (justify right))
     )
-    (property "Footprint" "" (id 2) (at 54.61 97.79 0)
+    (property "Footprint" "Capacitor_SMD:C_0201_0603Metric" (id 2) (at 54.61 97.79 0)
       (effects (font (size 1.27 1.27)) hide)
     )
@@
       (effects (font (size 1.27 1.27)) (justify right))
     )
-    (property "Footprint" "" (id 2) (at 67.31 99.06 0)
+    (property "Footprint" "Capacitor_SMD:C_0201_0603Metric" (id 2) (at 67.31 99.06 0)
       (effects (font (size 1.27 1.27)) hide)
     )
@@
       (effects (font (size 1.27 1.27)) (justify right))
     )
-    (property "Footprint" "" (id 2) (at 158.4452 97.79 0)
+    (property "Footprint" "Capacitor_SMD:C_0201_0603Metric" (id 2) (at 158.4452 97.79 0)
       (effects (font (size 1.27 1.27)) hide)
     )
@@
       (effects (font (size 1.27 1.27)) (justify right))
     )
-    (property "Footprint" "" (id 2) (at 78.74 99.06 0)
+    (property "Footprint" "Capacitor_SMD:C_0201_0603Metric" (id 2) (at 78.74 99.06 0)
       (effects (font (size 1.27 1.27)) hide)
     )
@@
       (effects (font (size 1.27 1.27)) (justify left))
     )
-    (property "Footprint" "" (id 2) (at 186.3852 105.41 0)
+    (property "Footprint" "Capacitor_SMD:C_0201_0603Metric" (id 2) (at 186.3852 105.41 0)
       (effects (font (size 1.27 1.27)) hide)
     )
@@
     (property "Reference" "C?" (id 0) (at 101.6 76.2 90))
     (property "Value" "C_Small" (id 1) (at 101.6 82.55 90))
-    (property "Footprint" "" (id 2) (at 101.6 78.74 0)
+    (property "Footprint" "Capacitor_SMD:C_0201_0603Metric" (id 2) (at 101.6 78.74 0)
       (effects (font (size 1.27 1.27)) hide)
     )
@@
       (effects (font (size 1.27 1.27)) (justify right))
     )
-    (property "Footprint" "" (id 2) (at 88.9 99.06 0)
-      (effects (font (size 1.27 1.27)) hide)
-    )
+    (property "Footprint" "Capacitor_SMD:C_0201_0603Metric" (id 2) (at 88.9 99.06 0)
+      (effects (font (size 1.27 1.27)) hide)
+    )
