File: DSAT_Telemetry_Board/DSAT_Telemetry_Board/LNA.kicad_sch (KiCad schematic)
At the start: 5 parts

Commit message: More footprints
Parts:
- C? (x3): footprint (none) -> Capacitor_SMD:C_0201_0603Metric
Changed lines of the file:
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@@
       (effects (font (size 1.27 1.27)) (justify left))
     )
-    (property "Footprint" "" (id 2) (at 185.1152 90.17 0)
+    (property "Footprint" "Capacitor_SMD:C_0201_0603Metric" (id 2) (at 185.1152 90.17 0)
       (effects (font (size 1.27 1.27)) hide)
     )
@@
     (property "Reference" "C?" (id 0) (at 120.65 96.52 90))
     (property "Value" "100pF" (id 1) (at 120.65 99.06 90))
-    (property "Footprint" "" (id 2) (at 124.46 105.1052 0)
+    (property "Footprint" "Capacitor_SMD:C_0201_0603Metric" (id 2) (at 124.46 105.1052 0)
       (effects (font (size 1.27 1.27)) hide)
     )
@@
     (property "Reference" "C?" (id 0) (at 173.99 96.52 90))
     (property "Value" "1.5nF" (id 1) (at 173.99 99.06 90))
-    (property "Footprint" "" (id 2) (at 177.8 105.1052 0)
+    (property "Footprint" "Capacitor_SMD:C_0201_0603Metric" (id 2) (at 177.8 105.1052 0)
       (effects (font (size 1.27 1.27)) hide)
     )

Commit message: RX_SWitch, test points
Parts:
- C? (x3): footprint Capacitor_SMD:C_0201_0603Metric -> Capacitor_SMD:C_0402_1005Metric_Pad0.74x0.62mm_HandSolder
- L?: footprint (none) -> Inductor_SMD:L_0402_1005Metric_Pad0.77x0.64mm_HandSolder
Changed lines of the file:
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@@
     (effects (font (size 1.27 1.27)) (justify left))
   )
-  (symbol (lib_id "DSAT_Telemetry_Libraries:PSA4-5043+") (at 140.97 96.52 0) (unit 1)
+  (symbol (lib_id "DSAT_Telemetry_Libraries:PSA4-5043+") (at 140.97 96.52 0)
     (in_bom yes) (on_board yes) (fields_autoplaced)
     (property "Reference" "U?" (id 0) (at 140.97 96.52 0))
@@
     (pin "4")
   )
-  (symbol (lib_id "power:GND") (at 140.97 124.46 0) (unit 1)
+  (symbol (lib_id "power:GND") (at 140.97 124.46 0)
     (in_bom yes) (on_board yes) (fields_autoplaced)
     (property "Reference" "#PWR?" (id 0) (at 140.97 130.81 0)
@@
     (pin "1")
   )
-  (symbol (lib_id "Device:L") (at 161.29 93.98 0) (unit 1)
+  (symbol (lib_id "Device:L") (at 161.29 93.98 0)
     (in_bom yes) (on_board yes) (fields_autoplaced)
     (property "Reference" "L?" (id 0) (at 162.56 92.7099 0)
@@
       (effects (font (size 1.27 1.27)) (justify left))
     )
-    (property "Footprint" "" (id 2) (at 161.29 93.98 0)
+    (property "Footprint" "Inductor_SMD:L_0402_1005Metric_Pad0.77x0.64mm_HandSolder" (id 2) (at 161.29 93.98 0)
       (effects (font (size 1.27 1.27)) hide)
     )
@@
     (pin "2")
   )
-  (symbol (lib_id "power:+3.3V") (at 184.15 78.74 0) (unit 1)
+  (symbol (lib_id "power:+3.3V") (at 184.15 78.74 0)
     (in_bom yes) (on_board yes) (fields_autoplaced)
     (property "Reference" "#PWR?" (id 0) (at 184.15 82.55 0)
@@
     (pin "1")
   )
-  (symbol (lib_id "Device:C") (at 184.15 86.36 0) (unit 1)
+  (symbol (lib_id "Device:C") (at 184.15 86.36 0)
     (in_bom yes) (on_board yes) (fields_autoplaced)
     (property "Reference" "C?" (id 0) (at 187.96 85.0899 0)
@@
       (effects (font (size 1.27 1.27)) (justify left))
     )
-    (property "Footprint" "Capacitor_SMD:C_0201_0603Metric" (id 2) (at 185.1152 90.17 0)
+    (property "Footprint" "Capacitor_SMD:C_0402_1005Metric_Pad0.74x0.62mm_HandSolder" (id 2) (at 185.1152 90.17 0)
       (effects (font (size 1.27 1.27)) hide)
     )
@@
     (pin "2")
   )
-  (symbol (lib_id "Device:C") (at 120.65 104.14 90) (mirror x) (unit 1)
+  (symbol (lib_id "Device:C") (at 120.65 104.14 90) (mirror x)
     (in_bom yes) (on_board yes) (fields_autoplaced)
     (property "Reference" "C?" (id 0) (at 120.65 96.52 90))
     (property "Value" "100pF" (id 1) (at 120.65 99.06 90))
-    (property "Footprint" "Capacitor_SMD:C_0201_0603Metric" (id 2) (at 124.46 105.1052 0)
+    (property "Footprint" "Capacitor_SMD:C_0402_1005Metric_Pad0.74x0.62mm_HandSolder" (id 2) (at 124.46 105.1052 0)
       (effects (font (size 1.27 1.27)) hide)
     )
@@
     (pin "2")
   )
-  (symbol (lib_id "power:GND") (at 184.15 90.17 0) (unit 1)
+  (symbol (lib_id "power:GND") (at 184.15 90.17 0)
     (in_bom yes) (on_board yes) (fields_autoplaced)
     (property "Reference" "#PWR?" (id 0) (at 184.15 96.52 0)
@@
     (pin "1")
   )
-  (symbol (lib_id "Device:C") (at 173.99 104.14 90) (mirror x) (unit 1)
+  (symbol (lib_id "Device:C") (at 173.99 104.14 90) (mirror x)
     (in_bom yes) (on_board yes) (fields_autoplaced)
     (property "Reference" "C?" (id 0) (at 173.99 96.52 90))
     (property "Value" "1.5nF" (id 1) (at 173.99 99.06 90))
-    (property "Footprint" "Capacitor_SMD:C_0201_0603Metric" (id 2) (at 177.8 105.1052 0)
+    (property "Footprint" "Capacitor_SMD:C_0402_1005Metric_Pad0.74x0.62mm_HandSolder" (id 2) (at 177.8 105.1052 0)
       (effects (font (size 1.27 1.27)) hide)
     )

Commit message: RX_SWitch, test points
Parts:
- gave numbers to parts that had none: 5
Connections:
- net Antenna renamed TX_LNA
Changed lines of the file:
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@@
     (effects (font (size 1.27 1.27)) (justify right))
   )
-  (hierarchical_label "Antenna" (shape input) (at 193.04 104.14 0)
+  (hierarchical_label "TX_LNA" (shape input) (at 193.04 104.14 0)
     (effects (font (size 1.27 1.27)) (justify left))
   )
-  (symbol (lib_id "DSAT_Telemetry_Libraries:PSA4-5043+") (at 140.97 96.52 0)
+  (symbol (lib_id "DSAT_Telemetry_Libraries:PSA4-5043+") (at 140.97 96.52 0) (unit 1)
     (in_bom yes) (on_board yes) (fields_autoplaced)
-    (property "Reference" "U?" (id 0) (at 140.97 96.52 0))
+    (property "Reference" "U7" (id 0) (at 140.97 96.52 0))
     (property "Value" "PSA4-5043+" (id 1) (at 140.97 99.06 0))
     (property "Footprint" "Package_TO_SOT_SMD:SOT-343_SC-70-4_Handsoldering" (id 2) (at 142.24 116.84 0)
@@
     (pin "4")
   )
-  (symbol (lib_id "power:GND") (at 140.97 124.46 0)
+  (symbol (lib_id "power:GND") (at 140.97 124.46 0) (unit 1)
     (in_bom yes) (on_board yes) (fields_autoplaced)
-    (property "Reference" "#PWR?" (id 0) (at 140.97 130.81 0)
+    (property "Reference" "#PWR0141" (id 0) (at 140.97 130.81 0)
       (effects (font (size 1.27 1.27)) hide)
     )
@@
     (pin "1")
   )
-  (symbol (lib_id "Device:L") (at 161.29 93.98 0)
+  (symbol (lib_id "Device:L") (at 161.29 93.98 0) (unit 1)
     (in_bom yes) (on_board yes) (fields_autoplaced)
-    (property "Reference" "L?" (id 0) (at 162.56 92.7099 0)
+    (property "Reference" "L4" (id 0) (at 162.56 92.7099 0)
       (effects (font (size 1.27 1.27)) (justify left))
     )
@@
     (pin "2")
   )
-  (symbol (lib_id "power:+3.3V") (at 184.15 78.74 0)
+  (symbol (lib_id "power:+3.3V") (at 184.15 78.74 0) (unit 1)
     (in_bom yes) (on_board yes) (fields_autoplaced)
-    (property "Reference" "#PWR?" (id 0) (at 184.15 82.55 0)
+    (property "Reference" "#PWR0140" (id 0) (at 184.15 82.55 0)
       (effects (font (size 1.27 1.27)) hide)
     )
@@
     (pin "1")
   )
-  (symbol (lib_id "Device:C") (at 184.15 86.36 0)
+  (symbol (lib_id "Device:C") (at 184.15 86.36 0) (unit 1)
     (in_bom yes) (on_board yes) (fields_autoplaced)
-    (property "Reference" "C?" (id 0) (at 187.96 85.0899 0)
+    (property "Reference" "C29" (id 0) (at 187.96 85.0899 0)
       (effects (font (size 1.27 1.27)) (justify left))
     )
@@
     (pin "2")
   )
-  (symbol (lib_id "Device:C") (at 120.65 104.14 90) (mirror x)
+  (symbol (lib_id "Device:C") (at 120.65 104.14 90) (mirror x) (unit 1)
     (in_bom yes) (on_board yes) (fields_autoplaced)
-    (property "Reference" "C?" (id 0) (at 120.65 96.52 90))
+    (property "Reference" "C27" (id 0) (at 120.65 96.52 90))
     (property "Value" "100pF" (id 1) (at 120.65 99.06 90))
     (property "Footprint" "Capacitor_SMD:C_0402_1005Metric_Pad0.74x0.62mm_HandSolder" (id 2) (at 124.46 105.1052 0)
@@
     (pin "2")
   )
-  (symbol (lib_id "power:GND") (at 184.15 90.17 0)
+  (symbol (lib_id "power:GND") (at 184.15 90.17 0) (unit 1)
     (in_bom yes) (on_board yes) (fields_autoplaced)
-    (property "Reference" "#PWR?" (id 0) (at 184.15 96.52 0)
+    (property "Reference" "#PWR0142" (id 0) (at 184.15 96.52 0)
       (effects (font (size 1.27 1.27)) hide)
     )
@@
     (pin "1")
   )
-  (symbol (lib_id "Device:C") (at 173.99 104.14 90) (mirror x)
+  (symbol (lib_id "Device:C") (at 173.99 104.14 90) (mirror x) (unit 1)
     (in_bom yes) (on_board yes) (fields_autoplaced)
-    (property "Reference" "C?" (id 0) (at 173.99 96.52 90))
+    (property "Reference" "C28" (id 0) (at 173.99 96.52 90))
     (property "Value" "1.5nF" (id 1) (at 173.99 99.06 90))
     (property "Footprint" "Capacitor_SMD:C_0402_1005Metric_Pad0.74x0.62mm_HandSolder" (id 2) (at 177.8 105.1052 0)
