File: DSAT_Telemetry_Board/DSAT_Telemetry_Board/RX_Switch.kicad_sch (KiCad schematic)
At the start: 6 parts

Commit message: RX_SWitch, test points
Parts:
- gave numbers to parts that had none: 6
Connections:
- net RX: now also IC1.3 (RF2); no longer IC1.1 (RF1)
- net TX_LNA: now also IC1.1 (RF1); no longer IC1.3 (RF2)
Changed lines of the file:
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@@
     (effects (font (size 1.27 1.27)) (justify left bottom))
+  )
+  (hierarchical_label "RX" (shape input) (at 175.26 107.95 0)
+    (effects (font (size 1.27 1.27)) (justify left))
   )
   (hierarchical_label "TX_En" (shape input) (at 144.78 107.95 180)
@@
     (effects (font (size 1.27 1.27)) (justify right))
   )
-  (hierarchical_label "RX" (shape input) (at 175.26 102.87 0)
+  (hierarchical_label "TX_LNA" (shape input) (at 175.26 102.87 0)
     (effects (font (size 1.27 1.27)) (justify left))
   )
-  (hierarchical_label "TX_LNA" (shape input) (at 175.26 107.95 0)
-    (effects (font (size 1.27 1.27)) (justify left))
-  )
-  (symbol (lib_id "Device:C_Small") (at 123.19 110.49 180)
+  (symbol (lib_id "Device:C_Small") (at 123.19 110.49 180) (unit 1)
     (in_bom yes) (on_board yes)
-    (property "Reference" "C?" (id 0) (at 125.73 109.2135 0)
+    (property "Reference" "C33" (id 0) (at 125.73 109.2135 0)
       (effects (font (size 1.27 1.27)) (justify right))
     )
@@
     (pin "2")
   )
-  (symbol (lib_id "power:GND") (at 175.26 105.41 90) (mirror x)
+  (symbol (lib_id "power:GND") (at 175.26 105.41 90) (mirror x) (unit 1)
     (in_bom yes) (on_board yes) (fields_autoplaced)
-    (property "Reference" "#PWR?" (id 0) (at 181.61 105.41 0)
+    (property "Reference" "#PWR0150" (id 0) (at 181.61 105.41 0)
       (effects (font (size 1.27 1.27)) hide)
     )
@@
     (pin "1")
   )
-  (symbol (lib_id "Device:L") (at 118.11 105.41 90)
+  (symbol (lib_id "Device:L") (at 118.11 105.41 90) (unit 1)
     (in_bom yes) (on_board yes) (fields_autoplaced)
-    (property "Reference" "L?" (id 0) (at 118.11 99.06 90))
+    (property "Reference" "L6" (id 0) (at 118.11 99.06 90))
     (property "Value" "36nH" (id 1) (at 118.11 101.6 90))
     (property "Footprint" "Inductor_SMD:L_0402_1005Metric_Pad0.77x0.64mm_HandSolder" (id 2) (at 118.11 105.41 0)
@@
     (pin "2")
   )
-  (symbol (lib_id "power:GND") (at 111.76 115.57 0) (mirror y)
+  (symbol (lib_id "power:GND") (at 111.76 115.57 0) (mirror y) (unit 1)
     (in_bom yes) (on_board yes) (fields_autoplaced)
-    (property "Reference" "#PWR?" (id 0) (at 111.76 121.92 0)
+    (property "Reference" "#PWR0148" (id 0) (at 111.76 121.92 0)
       (effects (font (size 1.27 1.27)) hide)
     )
@@
     (pin "1")
   )
-  (symbol (lib_id "power:GND") (at 123.19 115.57 0) (mirror y)
+  (symbol (lib_id "power:GND") (at 123.19 115.57 0) (mirror y) (unit 1)
     (in_bom yes) (on_board yes) (fields_autoplaced)
-    (property "Reference" "#PWR?" (id 0) (at 123.19 121.92 0)
+    (property "Reference" "#PWR0149" (id 0) (at 123.19 121.92 0)
       (effects (font (size 1.27 1.27)) hide)
     )
@@
     (pin "1")
   )
-  (symbol (lib_id "CG2409X3-C2:CG2409X3-C2") (at 175.26 102.87 0) (mirror y)
+  (symbol (lib_id "CG2409X3-C2:CG2409X3-C2") (at 175.26 102.87 0) (mirror y) (unit 1)
     (in_bom yes) (on_board yes) (fields_autoplaced)
-    (property "Reference" "IC?" (id 0) (at 160.02 95.25 0))
+    (property "Reference" "IC1" (id 0) (at 160.02 95.25 0))
     (property "Value" "CG2409X3-C2" (id 1) (at 160.02 97.79 0))
     (property "Footprint" "CG2409X3-C2:SON50P150X150X40-7N" (id 2) (at 148.59 100.33 0)
@@
     (pin "7")
   )
-  (symbol (lib_id "Device:L") (at 105.41 105.41 90)
+  (symbol (lib_id "Device:L") (at 105.41 105.41 90) (unit 1)
     (in_bom yes) (on_board yes) (fields_autoplaced)
-    (property "Reference" "L?" (id 0) (at 105.41 99.06 90))
+    (property "Reference" "L5" (id 0) (at 105.41 99.06 90))
     (property "Value" "22nH" (id 1) (at 105.41 101.6 90))
     (property "Footprint" "Inductor_SMD:L_0402_1005Metric_Pad0.77x0.64mm_HandSolder" (id 2) (at 105.41 105.41 0)
@@
     (pin "2")
   )
-  (symbol (lib_id "Device:C_Small") (at 111.76 110.49 180)
+  (symbol (lib_id "Device:C_Small") (at 111.76 110.49 180) (unit 1)
     (in_bom yes) (on_board yes)
-    (property "Reference" "C?" (id 0) (at 114.3 109.2135 0)
+    (property "Reference" "C32" (id 0) (at 114.3 109.2135 0)
       (effects (font (size 1.27 1.27)) (justify right))
     )
@@
     (pin "2")
   )
-  (symbol (lib_id "power:GND") (at 160.02 125.73 0)
+  (symbol (lib_id "power:GND") (at 160.02 125.73 0) (unit 1)
     (in_bom yes) (on_board yes) (fields_autoplaced)
-    (property "Reference" "#PWR?" (id 0) (at 160.02 132.08 0)
+    (property "Reference" "#PWR0147" (id 0) (at 160.02 132.08 0)
       (effects (font (size 1.27 1.27)) hide)
     )
@@
     (pin "1")
   )
-  (symbol (lib_id "Device:L") (at 129.54 105.41 90)
+  (symbol (lib_id "Device:L") (at 129.54 105.41 90) (unit 1)
     (in_bom yes) (on_board yes) (fields_autoplaced)
-    (property "Reference" "L?" (id 0) (at 129.54 99.06 90))
+    (property "Reference" "L7" (id 0) (at 129.54 99.06 90))
     (property "Value" "30nH" (id 1) (at 129.54 101.6 90))
     (property "Footprint" "Inductor_SMD:L_0402_1005Metric_Pad0.77x0.64mm_HandSolder" (id 2) (at 129.54 105.41 0)
