File: DSAT_Telemetry_Board/DSAT_Telemetry_Board/Watchdog_Timer_sch.kicad_sch (KiCad schematic)
At the start: 4 parts

Commit message: More footprints
Parts:
- C? (x2): footprint Capacitor_SMD:C_0201_0603Metric_Pad0.64x0.40mm_HandSolder -> Capacitor_SMD:C_0201_0603Metric
- R?: footprint (none) -> Resistor_SMD:R_0805_2012Metric
Changed lines of the file:
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@@
       (effects (font (size 1.27 1.27)) (justify right))
     )
-    (property "Footprint" "Capacitor_SMD:C_0201_0603Metric_Pad0.64x0.40mm_HandSolder" (id 2) (at 108.2548 77.47 0)
+    (property "Footprint" "Capacitor_SMD:C_0201_0603Metric" (id 2) (at 108.2548 77.47 0)
       (effects (font (size 1.27 1.27)) hide)
     )
-    (property "Datasheet" "~" (id 3) (at 109.22 81.28 0)
+    (property "Datasheet" "https://www.digikey.com/en/products/detail/murata-electronics/GRM033C80J123KE01D/2543438" (id 3) (at 109.22 81.28 0)
       (effects (font (size 1.27 1.27)) hide)
     )
@@
       (effects (font (size 1.27 1.27)) (justify right))
     )
-    (property "Footprint" "Capacitor_SMD:C_0201_0603Metric_Pad0.64x0.40mm_HandSolder" (id 2) (at 98.0948 77.47 0)
+    (property "Footprint" "Capacitor_SMD:C_0201_0603Metric" (id 2) (at 98.0948 77.47 0)
       (effects (font (size 1.27 1.27)) hide)
     )
-    (property "Datasheet" "~" (id 3) (at 99.06 81.28 0)
+    (property "Datasheet" "https://www.digikey.com/en/products/detail/murata-electronics/GRM033C80J123KE01D/2543438" (id 3) (at 99.06 81.28 0)
       (effects (font (size 1.27 1.27)) hide)
     )
@@
       (effects (font (size 1.27 1.27)) (justify right))
     )
-    (property "Footprint" "" (id 2) (at 110.998 60.96 90)
+    (property "Footprint" "Resistor_SMD:R_0805_2012Metric" (id 2) (at 110.998 60.96 90)
       (effects (font (size 1.27 1.27)) hide)
     )
-    (property "Datasheet" "~" (id 3) (at 109.22 60.96 0)
+    (property "Datasheet" "https://www.digikey.com/en/products/detail/vishay-dale/M55342K06B100ERS3/2941800" (id 3) (at 109.22 60.96 0)
       (effects (font (size 1.27 1.27)) hide)
     )

Commit message: RX_SWitch, test points
Parts:
- C? (x2): footprint Capacitor_SMD:C_0201_0603Metric -> Capacitor_SMD:C_0402_1005Metric_Pad0.74x0.62mm_HandSolder
- R?: footprint Resistor_SMD:R_0805_2012Metric -> Resistor_SMD:R_0402_1005Metric_Pad0.72x0.64mm_HandSolder
Changed lines of the file:
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@@
     (effects (font (size 1.27 1.27)) (justify left))
   )
-  (symbol (lib_id "Device:C") (at 109.22 81.28 180) (unit 1)
+  (symbol (lib_id "Device:C") (at 109.22 81.28 180)
     (in_bom yes) (on_board yes) (fields_autoplaced)
     (property "Reference" "C?" (id 0) (at 113.03 80.0099 0)
@@
       (effects (font (size 1.27 1.27)) (justify right))
     )
-    (property "Footprint" "Capacitor_SMD:C_0201_0603Metric" (id 2) (at 108.2548 77.47 0)
+    (property "Footprint" "Capacitor_SMD:C_0402_1005Metric_Pad0.74x0.62mm_HandSolder" (id 2) (at 108.2548 77.47 0)
       (effects (font (size 1.27 1.27)) hide)
     )
@@
     (pin "2")
   )
-  (symbol (lib_id "Device:C") (at 99.06 81.28 180) (unit 1)
+  (symbol (lib_id "Device:C") (at 99.06 81.28 180)
     (in_bom yes) (on_board yes)
     (property "Reference" "C?" (id 0) (at 102.87 80.01 0)
@@
       (effects (font (size 1.27 1.27)) (justify right))
     )
-    (property "Footprint" "Capacitor_SMD:C_0201_0603Metric" (id 2) (at 98.0948 77.47 0)
+    (property "Footprint" "Capacitor_SMD:C_0402_1005Metric_Pad0.74x0.62mm_HandSolder" (id 2) (at 98.0948 77.47 0)
       (effects (font (size 1.27 1.27)) hide)
     )
@@
     (pin "2")
   )
-  (symbol (lib_id "power:+3.3V") (at 143.51 52.07 0) (unit 1)
+  (symbol (lib_id "power:+3.3V") (at 143.51 52.07 0)
     (in_bom yes) (on_board yes) (fields_autoplaced)
     (property "Reference" "#PWR?" (id 0) (at 143.51 55.88 0)
@@
     (pin "1")
   )
-  (symbol (lib_id "Device:R") (at 109.22 60.96 180) (unit 1)
+  (symbol (lib_id "Device:R") (at 109.22 60.96 180)
     (in_bom yes) (on_board yes) (fields_autoplaced)
     (property "Reference" "R?" (id 0) (at 111.76 59.6899 0)
@@
       (effects (font (size 1.27 1.27)) (justify right))
     )
-    (property "Footprint" "Resistor_SMD:R_0805_2012Metric" (id 2) (at 110.998 60.96 90)
+    (property "Footprint" "Resistor_SMD:R_0402_1005Metric_Pad0.72x0.64mm_HandSolder" (id 2) (at 110.998 60.96 90)
       (effects (font (size 1.27 1.27)) hide)
     )
@@
     (pin "2")
   )
-  (symbol (lib_id "Watchdog_Timer:Watchdog_Timer") (at 129.54 64.77 0) (unit 1)
+  (symbol (lib_id "Watchdog_Timer:Watchdog_Timer") (at 129.54 64.77 0)
     (in_bom yes) (on_board yes) (fields_autoplaced)
     (property "Reference" "U?" (id 0) (at 129.54 62.23 0))
@@
     (pin "")
   )
-  (symbol (lib_id "power:GND") (at 119.38 95.25 0) (unit 1)
+  (symbol (lib_id "power:GND") (at 119.38 95.25 0)
     (in_bom yes) (on_board yes) (fields_autoplaced)
     (property "Reference" "#PWR?" (id 0) (at 119.38 101.6 0)

Commit message: RX_SWitch, test points
Parts:
- U8: renamed from U?; footprint (none) -> Package_SO:MSOP-8-1EP_3x3mm_P0.65mm_EP1.73x1.85mm
- gave numbers to parts that had none: 3
Changed lines of the file:
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@@
     (effects (font (size 1.27 1.27)) (justify left))
   )
-  (symbol (lib_id "Device:C") (at 109.22 81.28 180)
+  (symbol (lib_id "Device:C") (at 109.22 81.28 180) (unit 1)
     (in_bom yes) (on_board yes) (fields_autoplaced)
-    (property "Reference" "C?" (id 0) (at 113.03 80.0099 0)
+    (property "Reference" "C31" (id 0) (at 113.03 80.0099 0)
       (effects (font (size 1.27 1.27)) (justify right))
     )
@@
     (pin "2")
   )
-  (symbol (lib_id "Device:C") (at 99.06 81.28 180)
+  (symbol (lib_id "Device:C") (at 99.06 81.28 180) (unit 1)
     (in_bom yes) (on_board yes)
-    (property "Reference" "C?" (id 0) (at 102.87 80.01 0)
+    (property "Reference" "C30" (id 0) (at 102.87 80.01 0)
       (effects (font (size 1.27 1.27)) (justify right))
     )
@@
     (pin "2")
   )
-  (symbol (lib_id "power:+3.3V") (at 143.51 52.07 0)
+  (symbol (lib_id "power:+3.3V") (at 143.51 52.07 0) (unit 1)
     (in_bom yes) (on_board yes) (fields_autoplaced)
-    (property "Reference" "#PWR?" (id 0) (at 143.51 55.88 0)
+    (property "Reference" "#PWR0143" (id 0) (at 143.51 55.88 0)
       (effects (font (size 1.27 1.27)) hide)
     )
@@
     (pin "1")
   )
-  (symbol (lib_id "Device:R") (at 109.22 60.96 180)
+  (symbol (lib_id "Device:R") (at 109.22 60.96 180) (unit 1)
     (in_bom yes) (on_board yes) (fields_autoplaced)
-    (property "Reference" "R?" (id 0) (at 111.76 59.6899 0)
+    (property "Reference" "R11" (id 0) (at 111.76 59.6899 0)
       (effects (font (size 1.27 1.27)) (justify right))
     )
@@
     (pin "2")
   )
-  (symbol (lib_id "Watchdog_Timer:Watchdog_Timer") (at 129.54 64.77 0)
+  (symbol (lib_id "Watchdog_Timer:Watchdog_Timer") (at 129.54 64.77 0) (unit 1)
     (in_bom yes) (on_board yes) (fields_autoplaced)
-    (property "Reference" "U?" (id 0) (at 129.54 62.23 0))
+    (property "Reference" "U8" (id 0) (at 129.54 62.23 0))
     (property "Value" "Watchdog_Timer" (id 1) (at 129.54 64.77 0))
-    (property "Footprint" "" (id 2) (at 129.54 64.77 0)
+    (property "Footprint" "Package_SO:MSOP-8-1EP_3x3mm_P0.65mm_EP1.73x1.85mm" (id 2) (at 129.54 64.77 0)
       (effects (font (size 1.27 1.27)) hide)
     )
-    (property "Datasheet" "" (id 3) (at 129.54 64.77 0)
+    (property "Datasheet" "https://www.ablic.com/en/doc/datasheet/watchdog_timer/S1410_1411_E.pdf" (id 3) (at 129.54 64.77 0)
       (effects (font (size 1.27 1.27)) hide)
     )
@@
     (pin "")
   )
-  (symbol (lib_id "power:GND") (at 119.38 95.25 0)
+  (symbol (lib_id "power:GND") (at 119.38 95.25 0) (unit 1)
     (in_bom yes) (on_board yes) (fields_autoplaced)
-    (property "Reference" "#PWR?" (id 0) (at 119.38 101.6 0)
+    (property "Reference" "#PWR0144" (id 0) (at 119.38 101.6 0)
       (effects (font (size 1.27 1.27)) hide)
     )

Commit message: Added Watchdog Timer Footprint
Added custom footprint for watchdog timer
Parts:
- U8: footprint Package_SO:MSOP-8-1EP_3x3mm_P0.65mm_EP1.73x1.85mm -> Watchdog_Footprints:Watchdog_Timer
Connections:
- net +3V3: now also U8.8 (VDD); no longer U8. (~{WDO})
- net GND: now also U8.4 (VSS), U8.9 (GND); no longer U8. (~{WDO})
- net WDI: now also U8.7 (WDI); no longer U8. (~{WDO})
- net WEN: now also U8.5 (WEN); no longer U8. (~{WDO})
- net ~{WDO}: now also U8.6 (~{WDO}); no longer U8. (~{WDO})
- net ~{W}/T: now also U8.1 (~{RST}); no longer U8. (~{WDO})
- net at C31.2: now also U8.3 (CWDT); no longer U8. (~{WDO})
- net at C30.2: now also U8.2 (CPOR); no longer U8. (~{WDO})
Changed lines of the file:
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@@
+    (stroke (width 0) (type default) (color 0 0 0 0))
+  )
+  (wire (pts (xy 119.38 90.17) (xy 129.54 90.17))
     (stroke (width 0) (type default) (color 0 0 0 0))
   )
@@
   )
   (wire (pts (xy 143.51 69.85) (xy 139.7 69.85))
+    (stroke (width 0) (type default) (color 0 0 0 0))
+  )
+  (wire (pts (xy 129.54 83.82) (xy 129.54 90.17))
     (stroke (width 0) (type default) (color 0 0 0 0))
   )
@@
     (property "Reference" "U8" (id 0) (at 129.54 62.23 0))
     (property "Value" "Watchdog_Timer" (id 1) (at 129.54 64.77 0))
-    (property "Footprint" "Package_SO:MSOP-8-1EP_3x3mm_P0.65mm_EP1.73x1.85mm" (id 2) (at 129.54 64.77 0)
+    (property "Footprint" "Watchdog_Footprints:Watchdog_Timer" (id 2) (at 129.54 64.77 0)
       (effects (font (size 1.27 1.27)) hide)
     )
@@
       (effects (font (size 1.27 1.27)) hide)
     )
-    (pin "")
-    (pin "")
-    (pin "")
-    (pin "")
-    (pin "")
-    (pin "")
-    (pin "")
-    (pin "")
+    (pin "1")
+    (pin "2")
+    (pin "3")
+    (pin "4")
+    (pin "5")
+    (pin "6")
+    (pin "7")
+    (pin "8")
+    (pin "9")
   )
   (symbol (lib_id "power:GND") (at 119.38 95.25 0) (unit 1)

Commit message: Fixed PCB
Added new voltage regulator, reorganized everything, added new lines, fixed most DRC issues. Added ground and power pours. Added more vias.
Connections:
- net +3V3 renamed +3.3V
- net ~{W}/T renamed ~{RST}
Changed lines of the file:
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@@
 (kicad_sch (version 20211123) (generator eeschema)
   (paper "A4")
-  (junction (at 143.51 54.61) (diameter 0) (color 0 0 0 0)
+  (junction (at 109.22 90.17) (diameter 0) (color 0 0 0 0)
   )
-  (junction (at 109.22 90.17) (diameter 0) (color 0 0 0 0)
+  (junction (at 147.32 50.8) (diameter 0) (color 0 0 0 0)
   )
   (junction (at 119.38 90.17) (diameter 0) (color 0 0 0 0)
@@
     (stroke (width 0) (type default) (color 0 0 0 0))
   )
+  (wire (pts (xy 147.32 69.85) (xy 139.7 69.85))
+    (stroke (width 0) (type default) (color 0 0 0 0))
+  )
+  (wire (pts (xy 147.32 50.8) (xy 147.32 69.85))
+    (stroke (width 0) (type default) (color 0 0 0 0))
+  )
   (wire (pts (xy 99.06 90.17) (xy 99.06 85.09))
     (stroke (width 0) (type default) (color 0 0 0 0))
   )
-  (wire (pts (xy 143.51 54.61) (xy 109.22 54.61))
+  (wire (pts (xy 147.32 50.8) (xy 109.22 50.8))
     (stroke (width 0) (type default) (color 0 0 0 0))
   )
@@
     (stroke (width 0) (type default) (color 0 0 0 0))
   )
-  (wire (pts (xy 119.38 90.17) (xy 119.38 95.25))
+  (wire (pts (xy 109.22 50.8) (xy 109.22 57.15))
     (stroke (width 0) (type default) (color 0 0 0 0))
   )
-  (wire (pts (xy 143.51 54.61) (xy 143.51 69.85))
+  (wire (pts (xy 119.38 90.17) (xy 119.38 95.25))
     (stroke (width 0) (type default) (color 0 0 0 0))
   )
@@
     (stroke (width 0) (type default) (color 0 0 0 0))
   )
-  (wire (pts (xy 109.22 54.61) (xy 109.22 57.15))
-    (stroke (width 0) (type default) (color 0 0 0 0))
-  )
   (wire (pts (xy 109.22 90.17) (xy 119.38 90.17))
     (stroke (width 0) (type default) (color 0 0 0 0))
@@
     (stroke (width 0) (type default) (color 0 0 0 0))
   )
-  (wire (pts (xy 143.51 69.85) (xy 139.7 69.85))
-    (stroke (width 0) (type default) (color 0 0 0 0))
-  )
   (wire (pts (xy 129.54 83.82) (xy 129.54 90.17))
     (stroke (width 0) (type default) (color 0 0 0 0))
   )
   (wire (pts (xy 101.6 69.85) (xy 109.22 69.85))
-    (stroke (width 0) (type default) (color 0 0 0 0))
-  )
-  (wire (pts (xy 143.51 52.07) (xy 143.51 54.61))
     (stroke (width 0) (type default) (color 0 0 0 0))
   )
@@
     (effects (font (size 1.27 1.27)) (justify left bottom))
   )
-  (hierarchical_label "~{W}{slash}T" (shape input) (at 101.6 69.85 180)
+  (hierarchical_label "~{RST}" (shape input) (at 101.6 69.85 180)
     (effects (font (size 1.27 1.27)) (justify right))
   )
@@
   (hierarchical_label "~{WDO}" (shape input) (at 139.7 77.47 0)
     (effects (font (size 1.27 1.27)) (justify left))
+  )
+  (symbol (lib_id "power:+3.3V") (at 147.32 50.8 0) (mirror y) (unit 1)
+    (in_bom yes) (on_board yes) (fields_autoplaced)
+    (property "Reference" "#PWR0105" (id 0) (at 147.32 54.61 0)
+      (effects (font (size 1.27 1.27)) hide)
+    )
+    (property "Value" "+3.3V" (id 1) (at 147.32 45.72 0))
+    (property "Footprint" "" (id 2) (at 147.32 50.8 0)
+      (effects (font (size 1.27 1.27)) hide)
+    )
+    (property "Datasheet" "" (id 3) (at 147.32 50.8 0)
+      (effects (font (size 1.27 1.27)) hide)
+    )
+    (pin "1")
   )
   (symbol (lib_id "Device:C") (at 109.22 81.28 180) (unit 1)
@@
     (pin "2")
   )
-  (symbol (lib_id "power:+3.3V") (at 143.51 52.07 0) (unit 1)
-    (in_bom yes) (on_board yes) (fields_autoplaced)
-    (property "Reference" "#PWR0143" (id 0) (at 143.51 55.88 0)
-      (effects (font (size 1.27 1.27)) hide)
-    )
-    (property "Value" "+3.3V" (id 1) (at 143.51 46.99 0))
-    (property "Footprint" "" (id 2) (at 143.51 52.07 0)
-      (effects (font (size 1.27 1.27)) hide)
-    )
-    (property "Datasheet" "" (id 3) (at 143.51 52.07 0)
-      (effects (font (size 1.27 1.27)) hide)
-    )
-    (pin "1")
-  )
   (symbol (lib_id "Device:R") (at 109.22 60.96 180) (unit 1)
